Commit message: Added controller configuration file, bringup launch file (Currently uses hard-coded path to the console json), and the controller plugin for th moodel

File: model/PSM1.urdf.xacro (robot description, xacro)
@@ -3,4 +3,5 @@
   <!-- Macros -->
   <xacro:include filename="$(find dvrk_model)/model/psm.urdf.xacro"/>
+  <xacro:include filename="$(find dvrk_model)/ros2_control/psm_base.ros2_control.xacro"/>
   <link name="world"/>
   <xacro:psm_sca
@@ -8,3 +9,4 @@
       parent_link="world"
       xyz="-0.25 0.0 0.5" rpy="0.0 0.0 3.1415926"/>
+  <xacro:psm_base_ros2_control name="psm"/>
 </robot>

File: model/psm.base.urdf.xacro (robot description, xacro)
@@ -51,5 +51,5 @@
     <!-- link, all visual links mimic outer_pitch value -->
     <!-- joint 2-1: outer_pitch_1 -->
-    <joint name="outer_pitch_1" type="continuous">
+    <joint name="outer_pitch" type="continuous">
       <parent link="${prefix}outer_yaw_link"/>
       <child link="${prefix}outer_pitch_back_link"/>
@@ -78,5 +78,5 @@
       <axis xyz="0 0 1"/>
       <origin rpy="-1.5708 -1.5708 0" xyz="0 0.0295 0.4285"/>
-      <mimic joint="outer_pitch_1" multiplier="1"/>
+      <mimic joint="outer_pitch" multiplier="1"/>
     </joint>
     <!-- link 2-2: outer_pitch_front -->
@@ -101,5 +101,5 @@
       <axis xyz="0 0 1"/>
       <origin rpy="0 0 0" xyz="0.04178 0.15007 -0.0137"/>
-      <mimic joint="outer_pitch_1" multiplier="-1"/>
+      <mimic joint="outer_pitch" multiplier="-1"/>
     </joint>
     <!-- link 2-3: outer_pitch_bottom -->
@@ -124,5 +124,5 @@
       <axis xyz="0 0 1"/>
       <origin rpy="0 0 0" xyz="0.04209 0.18695 -0.02412"/>
-      <mimic joint="outer_pitch_1" multiplier="-1"/>
+      <mimic joint="outer_pitch" multiplier="-1"/>
     </joint>
     <!-- link 2-4: outer_pitch_top -->
@@ -147,5 +147,5 @@
       <axis xyz="0 0 1"/>
       <origin rpy="0 0 0" xyz="-0.520 0 -0.0155"/>
-      <mimic joint="outer_pitch_1" multiplier="1"/>
+      <mimic joint="outer_pitch" multiplier="1"/>
     </joint>
     <!-- link 2-5: outer_insertion -->
