Commit message: switch psm urdf to psm3

File: model/psm.urdf.xacro (robot description, xacro)
@@ -5,4 +5,6 @@
   <xacro:include filename="$(find dvrk_model)/model/psm.tool.sca.urdf.xacro"/>
   <xacro:include filename="$(find dvrk_model)/model/psm.tool.caudier.urdf.xacro"/>
+  <xacro:include filename="$(find dvrk_model)/model/psm.tool.caudier.blade.urdf.xacro"/>
+  <xacro:include filename="$(find dvrk_model)/model/psm.tool.sca.blade.urdf.xacro"/>
   <xacro:include filename="$(find dvrk_model)/model/psm.tool.snake.urdf.xacro"/>
   <!-- Macro for psm with snake -->
@@ -24,4 +26,21 @@
         prefix="${prefix}"/>
   </xacro:macro>
+  <!-- Macro for psm with sca -->
+  <xacro:macro name="psm_sca_blade" params="prefix parent_link xyz rpy">
+    <xacro:psm
+        prefix="${prefix}"
+        parent_link="${parent_link}"
+        xyz="${xyz}" rpy="${rpy}"/>
+    <xacro:psm_tool_sca_blade
+        prefix="${prefix}"/>
+  </xacro:macro>
+  <xacro:macro name="psm_caudier_blade" params="prefix parent_link xyz rpy">
+    <xacro:psm
+        prefix="${prefix}"
+        parent_link="${parent_link}"
+        xyz="${xyz}" rpy="${rpy}"/>
+    <xacro:psm_tool_caudier_blade
+        prefix="${prefix}"/>
+  </xacro:macro>
   <!-- Macro for psm with caudier -->
   <xacro:macro name="psm_caudier" params="prefix parent_link xyz rpy">
