Commit message: Added ccollision tags for the links and edited the ordering of links and made a continours chain that can be used in moveit for effective planning.

File: model/psm.base.urdf.xacro (robot description, xacro)
@@ -13,7 +13,13 @@
         <origin rpy="1.5708 0 3.1416" xyz="0.039 -0.40788 -0.07879"/>
         <geometry>
-          <mesh filename="package://dvrk_model/meshes/psm/psm_base.stl"/>
-        </geometry>
-      </visual>
+          <mesh filename="package://dvrk_model/meshes/psm/psm_base.dae"/>
+        </geometry>
+      </visual>
+      <collision>
+        <origin rpy="1.5708 0 3.1416" xyz="0.039 -0.40788 -0.07879"/>
+        <geometry>
+          <mesh filename="package://dvrk_model/meshes/psm/psm_base.dae"/>
+        </geometry>
+      </collision>
     </link>
     <!-- joint 1 -->
@@ -31,7 +37,13 @@
         <origin rpy="3.1416 0 1.5708" xyz="0.0125 0 0.5265"/>
         <geometry>
-          <mesh filename="package://dvrk_model/meshes/psm/outer_yaw.stl"/>
-        </geometry>
-      </visual>
+          <mesh filename="package://dvrk_model/meshes/psm/outer_yaw.dae"/>
+        </geometry>
+      </visual>
+      <collision>        <!-- <origin rpy="0 0 -1.5708" xyz="0.0125 0 0.1575"/> -->
+        <origin rpy="3.1416 0 1.5708" xyz="0.0125 0 0.5265"/>
+        <geometry>
+          <mesh filename="package://dvrk_model/meshes/psm/outer_yaw.dae"/>
+        </geometry>
+      </collision>
     </link>
     <!-- Note: I can not put visual link here as it's parallel -->
@@ -55,5 +67,5 @@
       <!-- <origin rpy="-1.5708 -1.5708 0" xyz="0 0.0295 0.1495"/> -->
       <origin rpy="-1.5708 -1.5708 0" xyz="0 0.0295 0.5185"/>
-      <mimic joint="outer_pitch" multiplier="1"/>
+      <!--<mimic joint="outer_pitch" multiplier="1"/> -->
     </joint>
     <!-- link 2-1: outer_pitch_back -->
@@ -62,7 +74,13 @@
         <origin rpy="0 0 -0.27129" xyz="0 0 0"/>
         <geometry>
-          <mesh filename="package://dvrk_model/meshes/psm/outer_pitch_back.stl"/>
-        </geometry>
-      </visual>
+          <mesh filename="package://dvrk_model/meshes/psm/outer_pitch_back.dae"/>
+        </geometry>
+      </visual>
+      <collision>
+        <origin rpy="0 0 -0.27129" xyz="0 0 0"/>
+        <geometry>
+          <mesh filename="package://dvrk_model/meshes/psm/outer_pitch_back.dae"/>
+        </geometry>
+      </collision>
     </link>
     <!-- joint 2-2: outer_pitch_2 -->
@@ -72,5 +90,5 @@
       <axis xyz="0 0 1"/>
       <origin rpy="-1.5708 -1.5708 0" xyz="0 0.0295 0.4285"/>
-      <mimic joint="outer_pitch" multiplier="1"/>
+      <mimic joint="outer_pitch_1" multiplier="1"/>
     </joint>
     <!-- link 2-2: outer_pitch_front -->
@@ -79,7 +97,13 @@
         <origin rpy="0 0 -0.27129" xyz="0 0 0"/>
         <geometry>
-          <mesh filename="package://dvrk_model/meshes/psm/outer_pitch_front.stl"/>
-        </geometry>
-      </visual>
+          <mesh filename="package://dvrk_model/meshes/psm/outer_pitch_front.dae"/>
+        </geometry>
+      </visual>
+      <collision>
+        <origin rpy="0 0 -0.27129" xyz="0 0 0"/>
+        <geometry>
+          <mesh filename="package://dvrk_model/meshes/psm/outer_pitch_front.dae"/>
+        </geometry>
+      </collision>
     </link>
     <!-- joint 2-3: outer_pitch_3 -->
@@ -89,5 +113,5 @@
       <axis xyz="0 0 1"/>
       <origin rpy="0 0 0" xyz="0.04178 0.15007 -0.0137"/>
-      <mimic joint="outer_pitch" multiplier="-1"/>
+      <mimic joint="outer_pitch_1" multiplier="-1"/>
     </joint>
     <!-- link 2-3: outer_pitch_bottom -->
@@ -96,7 +120,13 @@
         <origin rpy="0 -1.5708 0" xyz="0.009 0 0"/>
         <geometry>
-          <mesh filename="package://dvrk_model/meshes/psm/outer_pitch_bottom.stl"/>
-        </geometry>
-      </visual>
+          <mesh filename="package://dvrk_model/meshes/psm/outer_pitch_bottom.dae"/>
+        </geometry>
+      </visual>
+      <collision>
+        <origin rpy="0 -1.5708 0" xyz="0.009 0 0"/>
+        <geometry>
+          <mesh filename="package://dvrk_model/meshes/psm/outer_pitch_bottom.dae"/>
+        </geometry>
+      </collision>
     </link>
     <!-- joint 2-4: outer_pitch_4 -->
@@ -106,5 +136,5 @@
       <axis xyz="0 0 1"/>
       <origin rpy="0 0 0" xyz="0.04209 0.18695 -0.02412"/>
-      <mimic joint="outer_pitch" multiplier="-1"/>
+      <mimic joint="outer_pitch_1" multiplier="-1"/>
     </joint>
     <!-- link 2-4: outer_pitch_top -->
@@ -113,7 +143,13 @@
         <origin rpy="0 -1.5708 0" xyz="0.009 0 0"/>
         <geometry>
-          <mesh filename="package://dvrk_model/meshes/psm/outer_pitch_top.stl"/>
-        </geometry>
-      </visual>
+          <mesh filename="package://dvrk_model/meshes/psm/outer_pitch_top.dae"/>
+        </geometry>
+      </visual>
+      <collision>
+        <origin rpy="0 -1.5708 0" xyz="0.009 0 0"/>
+        <geometry>
+          <mesh filename="package://dvrk_model/meshes/psm/outer_pitch_top.dae"/>
+        </geometry>
+      </collision>
     </link>
     <!-- joint 2-5: outer_pitch_5 -->
@@ -123,5 +159,5 @@
       <axis xyz="0 0 1"/>
       <origin rpy="0 0 0" xyz="-0.520 0 -0.0155"/>
-      <mimic joint="outer_pitch" multiplier="1"/>
+      <mimic joint="outer_pitch_1" multiplier="1"/>
     </joint>
     <!-- link 2-5: outer_insertion -->
@@ -130,16 +166,23 @@
         <origin rpy="0 -1.5708 1.5708" xyz="0.02528 0.429 0"/>
         <geometry>
-          <mesh filename="package://dvrk_model/meshes/psm/outer_insertion.stl"/>
-        </geometry>
-      </visual>
+          <mesh filename="package://dvrk_model/meshes/psm/outer_insertion.dae"/>
+        </geometry>
+      </visual>
+      <collision>
+        <origin rpy="0 -1.5708 1.5708" xyz="0.02528 0.429 0"/>
+        <geometry>
+          <mesh filename="package://dvrk_model/meshes/psm/outer_insertion.dae"/>
+        </geometry>
+      </collision>
     </link>
     <!-- joint 3: insertion -->
     <joint name="outer_insertion" type="prismatic">
-      <!-- <parent link="${prefix}outer_insertion_link"/> -->
+      <parent link="${prefix}outer_insertion_link"/>
       <!-- <parent link="${prefix}psm_base_link"/> -->
-      <parent link="${prefix}outer_pitch_link"/>
+      <!--<parent link="${prefix}outer_pitch_link"/> -->
       <child link="${prefix}tool_main_link"/>
       <axis xyz="0 0 1"/>
-      <origin rpy="1.5708 0 0" xyz="0 0.4318 0"/>
+      <!--<origin rpy="1.5708 0 0" xyz="0 0.4318 0"/>-->
+      <origin rpy="1.5708 0 0" xyz="-0.040 0.282 0"/>
       <limit lower="0" upper="0.240" velocity=".4" effort="1000"/>
     </joint>
@@ -149,7 +192,13 @@
         <origin rpy="0 0 1.5708" xyz="0 0 0.041"/>
         <geometry>
-          <mesh filename="package://dvrk_model/meshes/psm/tool_main.stl"/>
-        </geometry>
-      </visual>
+          <mesh filename="package://dvrk_model/meshes/psm/tool_main.dae"/>
+        </geometry>
+      </visual>
+      <collision>
+        <origin rpy="0 0 1.5708" xyz="0 0 0.041"/>
+        <geometry>
+          <mesh filename="package://dvrk_model/meshes/psm/tool_main.dae"/>
+        </geometry>
+      </collision>
     </link>
     <!-- joint 4: Outer Roll -->
@@ -166,7 +215,13 @@
         <origin rpy="0 0 1.5708" xyz="0 0 -0.0091"/>
         <geometry>
-          <mesh filename="package://dvrk_model/meshes/psm/tool_wrist_link.stl"/>
-        </geometry>
-      </visual>
+          <mesh filename="package://dvrk_model/meshes/psm/tool_wrist_link.dae"/>
+        </geometry>
+      </visual>
+      <collision>
+        <origin rpy="0 0 1.5708" xyz="0 0 -0.0091"/>
+        <geometry>
+          <mesh filename="package://dvrk_model/meshes/psm/tool_wrist_link.dae"/>
+        </geometry>
+      </collision>
     </link>
     <!-- joint 4-1: outer roll shaft joint FIXED-->
@@ -182,7 +237,13 @@
         <origin rpy="1.5708 0 0" xyz="0 0.00401 0"/>
         <geometry>
-          <mesh filename="package://dvrk_model/meshes/psm/tool_wrist_shaft_link.stl"/>
-        </geometry>
-      </visual>
+          <mesh filename="package://dvrk_model/meshes/psm/tool_wrist_shaft_link.dae"/>
+        </geometry>
+      </visual>
+      <collision>
+        <origin rpy="1.5708 0 0" xyz="0 0.00401 0"/>
+        <geometry>
+          <mesh filename="package://dvrk_model/meshes/psm/tool_wrist_shaft_link.dae"/>
+        </geometry>
+      </collision>
     </link>
   </xacro:macro>

File: model/psm.tool.sca.urdf.xacro (robot description, xacro)
@@ -22,4 +22,11 @@
         </geometry>
       </visual>
+      <collision>
+        <!-- <origin rpy="0 3.1416 0" xyz="0 0 0"/> -->
+        <origin rpy="1.5708 3.1416 0" xyz="0.0051 0.0032 0"/>
+        <geometry>
+          <mesh filename="package://dvrk_model/meshes/psm/tool_wrist_sca_link.stl"/>
+        </geometry>
+      </collision>
     </link>
     <!-- joint 6: Outer wrist yaw joint -->
@@ -40,4 +47,10 @@
         </geometry>
       </visual>
+      <collision>
+        <origin rpy="0 0 0" xyz="0 -0.0002 -0.0025"/>
+        <geometry>
+          <mesh filename="package://dvrk_model/meshes/psm/tool_wrist_sca_shaft_link.stl"/>
+        </geometry>
+      </collision>
     </link>
     <!-- joint 7-0: Outer open angle 1  -->
@@ -57,4 +70,10 @@
         </geometry>
       </visual>
+      <collision>
+        <origin rpy="0 0 0" xyz="0 0 0"/>
+        <geometry>
+          <box size="0 0 0" />
+        </geometry>
+      </collision>
     </link>
     <!-- joint 7-1: Outer open angle 1  -->
@@ -75,4 +94,10 @@
         </geometry>
       </visual>
+      <collision>
+        <origin rpy="0 0 0" xyz="0 0 0"/>
+        <geometry>
+          <mesh filename="package://dvrk_model/meshes/psm/tool_wrist_sca_link_2.stl"/>
+        </geometry>
+      </collision>
     </link>
     <!-- joint 7-2: Outer open angle 2   -->
@@ -93,4 +118,10 @@
         </geometry>
       </visual>
+      <collision>
+        <origin rpy="0 3.1516 0" xyz="0 0 0"/>
+        <geometry>
+          <mesh filename="package://dvrk_model/meshes/psm/tool_wrist_sca_link_2.stl"/>
+        </geometry>
+      </collision>
     </link>
     <!-- tool tip -->

Commit message: Changed files to stl and removed the old code and trailing spaces.

File: model/psm.base.urdf.xacro (robot description, xacro)
@@ -13,5 +13,5 @@
         <origin rpy="1.5708 0 3.1416" xyz="0.039 -0.40788 -0.07879"/>
         <geometry>
-          <mesh filename="package://dvrk_model/meshes/psm/psm_base.dae"/>
+          <mesh filename="package://dvrk_model/meshes/psm/psm_base.stl"/>
         </geometry>
       </visual>
@@ -19,5 +19,5 @@
         <origin rpy="1.5708 0 3.1416" xyz="0.039 -0.40788 -0.07879"/>
         <geometry>
-          <mesh filename="package://dvrk_model/meshes/psm/psm_base.dae"/>
+          <mesh filename="package://dvrk_model/meshes/psm/psm_base.stl"/>
         </geometry>
       </collision>
@@ -37,5 +37,5 @@
         <origin rpy="3.1416 0 1.5708" xyz="0.0125 0 0.5265"/>
         <geometry>
-          <mesh filename="package://dvrk_model/meshes/psm/outer_yaw.dae"/>
+          <mesh filename="package://dvrk_model/meshes/psm/outer_yaw.stl"/>
         </geometry>
       </visual>
@@ -43,5 +43,5 @@
         <origin rpy="3.1416 0 1.5708" xyz="0.0125 0 0.5265"/>
         <geometry>
-          <mesh filename="package://dvrk_model/meshes/psm/outer_yaw.dae"/>
+          <mesh filename="package://dvrk_model/meshes/psm/outer_yaw.stl"/>
         </geometry>
       </collision>
@@ -50,14 +50,4 @@
     <!-- mechanism, so the outer_pitch_link does not have visual -->
     <!-- link, all visual links mimic outer_pitch value -->
-    <!-- joint 2: outer_pitch -->
-    <joint name="outer_pitch" type="revolute">
-      <parent link="${prefix}outer_yaw_link"/>
-      <child link="${prefix}outer_pitch_link"/>
-      <axis xyz="0 0 1"/>
-      <origin rpy="-1.5708 -1.5708 0" xyz="0 0 0"/>
-      <limit lower="-0.7854" upper="0.7854" velocity=".4" effort="1000"/>
-    </joint>
-    <!-- link 2: outer_pitch_link -->
-    <link name="${prefix}outer_pitch_link"/>
     <!-- joint 2-1: outer_pitch_1 -->
     <joint name="outer_pitch_1" type="continuous">
@@ -65,7 +55,5 @@
       <child link="${prefix}outer_pitch_back_link"/>
       <axis xyz="0 0 1"/>
-      <!-- <origin rpy="-1.5708 -1.5708 0" xyz="0 0.0295 0.1495"/> -->
       <origin rpy="-1.5708 -1.5708 0" xyz="0 0.0295 0.5185"/>
-      <!--<mimic joint="outer_pitch" multiplier="1"/> -->
     </joint>
     <!-- link 2-1: outer_pitch_back -->
@@ -74,11 +62,11 @@
         <origin rpy="0 0 -0.27129" xyz="0 0 0"/>
         <geometry>
-          <mesh filename="package://dvrk_model/meshes/psm/outer_pitch_back.dae"/>
-        </geometry>
-      </visual>
-      <collision>
-        <origin rpy="0 0 -0.27129" xyz="0 0 0"/>
-        <geometry>
-          <mesh filename="package://dvrk_model/meshes/psm/outer_pitch_back.dae"/>
+          <mesh filename="package://dvrk_model/meshes/psm/outer_pitch_back.stl"/>
+        </geometry>
+      </visual>
+      <collision>
+        <origin rpy="0 0 -0.27129" xyz="0 0 0"/>
+        <geometry>
+          <mesh filename="package://dvrk_model/meshes/psm/outer_pitch_back.stl"/>
         </geometry>
       </collision>
@@ -97,11 +85,11 @@
         <origin rpy="0 0 -0.27129" xyz="0 0 0"/>
         <geometry>
-          <mesh filename="package://dvrk_model/meshes/psm/outer_pitch_front.dae"/>
-        </geometry>
-      </visual>
-      <collision>
-        <origin rpy="0 0 -0.27129" xyz="0 0 0"/>
-        <geometry>
-          <mesh filename="package://dvrk_model/meshes/psm/outer_pitch_front.dae"/>
+          <mesh filename="package://dvrk_model/meshes/psm/outer_pitch_front.stl"/>
+        </geometry>
+      </visual>
+      <collision>
+        <origin rpy="0 0 -0.27129" xyz="0 0 0"/>
+        <geometry>
+          <mesh filename="package://dvrk_model/meshes/psm/outer_pitch_front.stl"/>
         </geometry>
       </collision>
@@ -120,11 +108,11 @@
         <origin rpy="0 -1.5708 0" xyz="0.009 0 0"/>
         <geometry>
-          <mesh filename="package://dvrk_model/meshes/psm/outer_pitch_bottom.dae"/>
-        </geometry>
-      </visual>
-      <collision>
-        <origin rpy="0 -1.5708 0" xyz="0.009 0 0"/>
-        <geometry>
-          <mesh filename="package://dvrk_model/meshes/psm/outer_pitch_bottom.dae"/>
+          <mesh filename="package://dvrk_model/meshes/psm/outer_pitch_bottom.stl"/>
+        </geometry>
+      </visual>
+      <collision>
+        <origin rpy="0 -1.5708 0" xyz="0.009 0 0"/>
+        <geometry>
+          <mesh filename="package://dvrk_model/meshes/psm/outer_pitch_bottom.stl"/>
         </geometry>
       </collision>
@@ -143,11 +131,11 @@
         <origin rpy="0 -1.5708 0" xyz="0.009 0 0"/>
         <geometry>
-          <mesh filename="package://dvrk_model/meshes/psm/outer_pitch_top.dae"/>
-        </geometry>
-      </visual>
-      <collision>
-        <origin rpy="0 -1.5708 0" xyz="0.009 0 0"/>
-        <geometry>
-          <mesh filename="package://dvrk_model/meshes/psm/outer_pitch_top.dae"/>
+          <mesh filename="package://dvrk_model/meshes/psm/outer_pitch_top.stl"/>
+        </geometry>
+      </visual>
+      <collision>
+        <origin rpy="0 -1.5708 0" xyz="0.009 0 0"/>
+        <geometry>
+          <mesh filename="package://dvrk_model/meshes/psm/outer_pitch_top.stl"/>
         </geometry>
       </collision>
@@ -166,5 +154,5 @@
         <origin rpy="0 -1.5708 1.5708" xyz="0.02528 0.429 0"/>
         <geometry>
-          <mesh filename="package://dvrk_model/meshes/psm/outer_insertion.dae"/>
+          <mesh filename="package://dvrk_model/meshes/psm/outer_insertion.stl"/>
         </geometry>
       </visual>
@@ -172,5 +160,5 @@
         <origin rpy="0 -1.5708 1.5708" xyz="0.02528 0.429 0"/>
         <geometry>
-          <mesh filename="package://dvrk_model/meshes/psm/outer_insertion.dae"/>
+          <mesh filename="package://dvrk_model/meshes/psm/outer_insertion.stl"/>
         </geometry>
       </collision>
@@ -179,9 +167,6 @@
     <joint name="outer_insertion" type="prismatic">
       <parent link="${prefix}outer_insertion_link"/>
-      <!-- <parent link="${prefix}psm_base_link"/> -->
-      <!--<parent link="${prefix}outer_pitch_link"/> -->
       <child link="${prefix}tool_main_link"/>
       <axis xyz="0 0 1"/>
-      <!--<origin rpy="1.5708 0 0" xyz="0 0.4318 0"/>-->
       <origin rpy="1.5708 0 0" xyz="-0.040 0.282 0"/>
       <limit lower="0" upper="0.240" velocity=".4" effort="1000"/>
@@ -192,5 +177,5 @@
         <origin rpy="0 0 1.5708" xyz="0 0 0.041"/>
         <geometry>
-          <mesh filename="package://dvrk_model/meshes/psm/tool_main.dae"/>
+          <mesh filename="package://dvrk_model/meshes/psm/tool_main.stl"/>
         </geometry>
       </visual>
@@ -198,5 +183,5 @@
         <origin rpy="0 0 1.5708" xyz="0 0 0.041"/>
         <geometry>
-          <mesh filename="package://dvrk_model/meshes/psm/tool_main.dae"/>
+          <mesh filename="package://dvrk_model/meshes/psm/tool_main.stl"/>
         </geometry>
       </collision>
@@ -215,5 +200,5 @@
         <origin rpy="0 0 1.5708" xyz="0 0 -0.0091"/>
         <geometry>
-          <mesh filename="package://dvrk_model/meshes/psm/tool_wrist_link.dae"/>
+          <mesh filename="package://dvrk_model/meshes/psm/tool_wrist_link.stl"/>
         </geometry>
       </visual>
@@ -221,5 +206,5 @@
         <origin rpy="0 0 1.5708" xyz="0 0 -0.0091"/>
         <geometry>
-          <mesh filename="package://dvrk_model/meshes/psm/tool_wrist_link.dae"/>
+          <mesh filename="package://dvrk_model/meshes/psm/tool_wrist_link.stl"/>
         </geometry>
       </collision>
@@ -237,5 +222,5 @@
         <origin rpy="1.5708 0 0" xyz="0 0.00401 0"/>
         <geometry>
-          <mesh filename="package://dvrk_model/meshes/psm/tool_wrist_shaft_link.dae"/>
+          <mesh filename="package://dvrk_model/meshes/psm/tool_wrist_shaft_link.stl"/>
         </geometry>
       </visual>
@@ -243,5 +228,5 @@
         <origin rpy="1.5708 0 0" xyz="0 0.00401 0"/>
         <geometry>
-          <mesh filename="package://dvrk_model/meshes/psm/tool_wrist_shaft_link.dae"/>
+          <mesh filename="package://dvrk_model/meshes/psm/tool_wrist_shaft_link.stl"/>
         </geometry>
       </collision>

Commit message: Added tool urdfs, modified PSM3.urdf.xacro and modified joint limits for shaft_roll

File: model/psm.base.urdf.xacro (robot description, xacro)
@@ -193,5 +193,5 @@
       <axis xyz="0 0 1"/>
       <origin rpy="0 0 0" xyz="0 0 0.4162"/>
-      <limit lower="-2.2689" upper="2.2689" velocity=".4" effort="1000"/>
+      <limit lower="-4.53786" upper="4.53786" velocity=".4" effort="1000"/>
     </joint>
     <!-- link 4: tool_wrist_link -->

File: model/psm.tool.caudier.blade.urdf.xacro (robot description, xacro)
@@ -62,10 +62,18 @@
       <visual>
         <origin rpy="0.0 0.0 0.0" xyz="0 0.0225 0"/>
+        <!-- <origin rpy="0.0 0.0 0.0" xyz="0 0 0"/> -->
         <geometry>
           <box size="0.005 0.045 0.001" />
         </geometry>
+        <!-- <geometry>
+          <mesh filename="package://dvrk_model/meshes/psm/knife.stl"/>
+        </geometry> -->
       </visual>
       <collision>
         <origin rpy="0.0 0.0 0.0" xyz="0 0.0225 0"/>
+        <!-- <origin rpy="0.0 0.0 0.0" xyz="0 0 0"/> -->
+        <!-- <geometry>
+          <mesh filename="package://dvrk_model/meshes/psm/knife.stl"/>
+        </geometry> -->
         <geometry>
           <box size="0.005  0.045 0.001" />
