Commit message: Addede tool with blade urdfs for caudier and sca

File: model/psm.tool.caudier.blade.urdf.xacro (robot description, xacro)
@@ -8,5 +8,5 @@
       <axis xyz="0 0 1"/>
       <origin rpy="-1.5708 -1.5708 0" xyz="0 0 0"/>
-      <limit lower="-1.5707" upper="1.5707" velocity=".4" effort="1000"/>
+      <limit lower="-1.39268" upper="1.39268" velocity=".4" effort="1000"/>
     </joint>
     <!-- link 5: tool_wrist_caudier_link -->
@@ -32,5 +32,5 @@
       <axis xyz="0 0 -1"/>
       <origin rpy="0.00 -1.5708 -1.5708" xyz="0.0091 0 0"/>
-      <limit lower="-1.5707" upper="1.5707" velocity=".4" effort="1000"/>
+      <limit lower="-1.39268" upper="1.39268" velocity=".4" effort="1000"/>
     </joint>
     <!-- link 6: tool_wrist_caudier_link_shaft -->

File: model/psm.tool.sca.blade.urdf.xacro (robot description, xacro)
@@ -9,5 +9,5 @@
       <axis xyz="0 0 1"/>
       <origin rpy="-1.5708 -1.5708 0" xyz="0 0 0"/>
-      <limit lower="-1.5707" upper="1.5707" velocity=".4" effort="1000"/>
+      <limit lower="-1.39268" upper="1.39268" velocity=".4" effort="1000"/>
     </joint>
     <!-- link 5: tool_wrist_sca_link -->
@@ -35,5 +35,5 @@
       <origin rpy="-1.5708 -1.5708 0" xyz="0.0091 0 0"/>
       <!-- +/- 80 deg -->
-      <limit lower="-1.3963" upper="1.3963" velocity=".4" effort="1000"/>
+      <limit lower="-1.39268" upper="1.39268" velocity=".4" effort="1000"/>
     </joint>
     <!-- link 6: tool_wrist_sca_shaft_link -->

Commit message: added blade model to the urdf

File: model/psm.tool.caudier.blade.urdf.xacro (robot description, xacro)
@@ -55,5 +55,5 @@
       <child link="${prefix}tool_wrist_caudier_ee_link_0"/>
       <!-- <axis xyz="0 1 0"/> -->
-      <origin rpy="0 0 0" xyz="0 0 0"/>
+      <origin rpy="-1.5708 0 0" xyz="0 0 0"/>
       <!-- <limit lower="0" upper="1.5707" velocity=".4" effort="1000"/> -->
     </joint>
@@ -61,22 +61,22 @@
     <link name="${prefix}tool_wrist_caudier_ee_link_0">
       <visual>
-        <origin rpy="0.0 0.0 0.0" xyz="0 0.0225 0"/>
-        <!-- <origin rpy="0.0 0.0 0.0" xyz="0 0 0"/> -->
+        <!-- <origin rpy="0.0 0.0 0.0" xyz="0 0.0225 0"/> -->
+        <origin rpy="0 0 0" xyz="0 0 0"/>
+        <!-- <geometry>
+          <box size="0.005 0.045 0.001" />
+        </geometry> -->
         <geometry>
-          <box size="0.005 0.045 0.001" />
+          <mesh filename="package://dvrk_model/meshes/psm/knife.STL"/>
+        </geometry>
+      </visual>
+      <collision>
+        <!-- <origin rpy="0.0 0.0 0.0" xyz="0 0.0225 0"/> -->
+        <origin rpy="0 0 0" xyz="0 0 0"/>
+        <geometry>
+          <mesh filename="package://dvrk_model/meshes/psm/knife.STL"/>
         </geometry>
         <!-- <geometry>
-          <mesh filename="package://dvrk_model/meshes/psm/knife.stl"/>
+          <box size="0.005  0.045 0.001" />
         </geometry> -->
-      </visual>
-      <collision>
-        <origin rpy="0.0 0.0 0.0" xyz="0 0.0225 0"/>
-        <!-- <origin rpy="0.0 0.0 0.0" xyz="0 0 0"/> -->
-        <!-- <geometry>
-          <mesh filename="package://dvrk_model/meshes/psm/knife.stl"/>
-        </geometry> -->
-        <geometry>
-          <box size="0.005  0.045 0.001" />
-        </geometry>
       </collision>
     </link>
@@ -85,5 +85,5 @@
       <parent link="${prefix}tool_wrist_caudier_ee_link_0"/>
       <child link="${prefix}tool_tip_link"/>
-      <origin rpy="-1.5708 0.0 0.0" xyz="0 0.045 0"/>
+      <origin rpy="0 0 0" xyz="0 0.045 0"/>
     </joint>
     <!-- link 6-3:  -->

Commit message: Moved tool tip to the tip of the blade

File: model/psm.tool.caudier.blade.urdf.xacro (robot description, xacro)
@@ -30,5 +30,5 @@
       <parent link="${prefix}tool_wrist_caudier_link"/>
       <child link="${prefix}tool_wrist_caudier_shaft_link"/>
-      <axis xyz="0 0 -1"/>
+      <axis xyz="0 0 1"/>
       <origin rpy="0.00 -1.5708 -1.5708" xyz="0.0091 0 0"/>
       <limit lower="-1.39268" upper="1.39268" velocity=".4" effort="1000"/>
@@ -83,7 +83,7 @@
     <!-- tool tip   -->
     <joint name="tool_wrist_caudier_ee" type="fixed">
-      <parent link="${prefix}tool_wrist_caudier_ee_link_0"/>
+      <parent link="${prefix}tool_wrist_caudier_shaft_link"/>
       <child link="${prefix}tool_tip_link"/>
-      <origin rpy="0 0 0" xyz="0 0.045 0"/>
+      <origin rpy="-1.5708 0 0" xyz="0 0.045 0.0025"/>
     </joint>
     <!-- link 6-3:  -->
