Commit message: switch wrist_roll to wrist_yaw

File: ros2_control/psm_base.ros2_control.xacro (robot description, xacro)
@@ -46,5 +46,5 @@
                 <state_interface name="velocity"/>
             </joint>
-            <joint name="outer_wrist_roll">
+            <joint name="outer_wrist_yaw">
                 <command_interface name="position">
                 <param name="min">-1.5707</param>
